File: PCB/_autosave-main_pcb.kicad_pcb (KiCad board)
At the start: 2 copper layers, 116.9 x 116.9 mm, 39 parts, among them P1 SEN, P2 SRV, P3 PWR, P4 LED, P5 M1, P6 M2, P7 CONN_02X03, P8 CONN_02X03, Q1 5LN01SP, U1 Teensy_3.1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

Commit message: Updated pcb layout for easier fabrication
Routing:
- net GND: track 454.5 -> 458.9 mm
- net /DIR1: track 88.4 -> 84.8 mm
- net /DIR2: track 93.9 -> 96.8 mm
- net /STEP2: track 91.7 -> 93.2 mm
- net /MISO: track 47.3 -> 48.0 mm
- net /MOSI: track 44.8 -> 44.2 mm
Other:
- outline, holes or cut-outs redrawn
- net class Default: via_dia 1 -> 1.6

Commit message: minor pcb and BOM adjustments
Routing:
- net /RadCS: vias 1 -> 2
Changed lines of the file:
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@@
     (thickness 1.6)
     (drawings 9)
-    (tracks 392)
+    (tracks 393)
     (zones 0)
     (modules 39)
@@
       (padsonsilk false)
       (subtractmaskfromsilk false)
-      (outputformat 1)
+      (outputformat 4)
       (mirror false)
       (drillshape 0)
@@
   (segment (start 132.08 119.38) (end 132.08 116.84) (width 0.25) (layer B.Cu) (net 37))
   (segment (start 140.97 128.27) (end 132.08 119.38) (width 0.25) (layer B.Cu) (net 37))
+  (via (at 140.97 123.19) (size 1.6) (drill 0.6) (layers F.Cu B.Cu) (net 45))
+  (segment (start 140.97 123.19) (end 144.78 123.19) (width 0.25) (layer B.Cu) (net 45) (status 800000))
   (segment (start 106.68 116.84) (end 106.68 120.65) (width 0.25) (layer B.Cu) (net 45))
-  (segment (start 140.97 123.19) (end 144.78 123.19) (width 0.25) (layer F.Cu) (net 45))
   (segment (start 137.16 127) (end 140.97 123.19) (width 0.25) (layer F.Cu) (net 45))
   (via (at 137.16 127) (size 1.6) (drill 0.6) (layers F.Cu B.Cu) (net 45))
