File: PCB/analogFilter.sch (KiCad schematic (older format))
At the start: 12 parts, among them U3 MCP6004

Commit message: Fixed some motor speed modelling errors
Parts:
- U3: footprint Housings_DIP:DIP-14_W7.62mm -> custom_footprints:DIP-14_W7.62mm_Socket
Changed lines of the file:
@@
-$Comp
-L MCP6004 U3
-U 1 1 5941D635
-P 4100 3650
-AR Path="/5941B2B4/5941D635" Ref="U3"  Part="1"
-AR Path="/5941F948/5941D635" Ref="U3"  Part="4"
-F 0 "U3" H 4150 3850 50  0000 C CNN
-F 1 "MCP6004" H 4250 3450 50  0000 C CNN
-F 2 "Housings_DIP:DIP-14_W7.62mm" H 4050 3750 50  0001 C CNN
-F 3 "" H 4150 3850 50  0000 C CNN
-	1    4100 3650
-	1    0    0    -1
-$EndComp
 $Comp
 L MCP6004 U3
@@
 F 0 "U3" H 5450 3750 50  0000 C CNN
 F 1 "MCP6004" H 5550 3350 50  0000 C CNN
-F 2 "Housings_DIP:DIP-14_W7.62mm" H 5350 3650 50  0001 C CNN
+F 2 "custom_footprints:DIP-14_W7.62mm_Socket" H 5350 3650 50  0001 C CNN
 F 3 "" H 5450 3750 50  0000 C CNN
 	2    5400 3550
@@
 F 0 "U3" H 6750 3650 50  0000 C CNN
 F 1 "MCP6004" H 6850 3250 50  0000 C CNN
-F 2 "Housings_DIP:DIP-14_W7.62mm" H 6650 3550 50  0001 C CNN
+F 2 "custom_footprints:DIP-14_W7.62mm_Socket" H 6650 3550 50  0001 C CNN
 F 3 "" H 6750 3650 50  0000 C CNN
 	3    6700 3450
@@
 AR Path="/5941B2B4/5941D64A" Ref="#PWR033"  Part="1"
 AR Path="/5941F948/5941D64A" Ref="#PWR038"  Part="1"
-F 0 "#PWR033" H 4000 3700 50  0001 C CNN
+F 0 "#PWR038" H 4000 3700 50  0001 C CNN
 F 1 "GND" H 4000 3800 50  0000 C CNN
 F 2 "" H 4000 3950 50  0000 C CNN
@@
 AR Path="/5941B2B4/5941D650" Ref="#PWR034"  Part="1"
 AR Path="/5941F948/5941D650" Ref="#PWR039"  Part="1"
-F 0 "#PWR034" H 5300 3600 50  0001 C CNN
+F 0 "#PWR039" H 5300 3600 50  0001 C CNN
 F 1 "GND" H 5300 3700 50  0000 C CNN
 F 2 "" H 5300 3850 50  0000 C CNN
@@
 AR Path="/5941B2B4/5941D656" Ref="#PWR035"  Part="1"
 AR Path="/5941F948/5941D656" Ref="#PWR040"  Part="1"
-F 0 "#PWR035" H 6600 3500 50  0001 C CNN
+F 0 "#PWR040" H 6600 3500 50  0001 C CNN
 F 1 "GND" H 6600 3600 50  0000 C CNN
 F 2 "" H 6600 3750 50  0000 C CNN
@@
 AR Path="/5941B2B4/5941E011" Ref="#PWR036"  Part="1"
 AR Path="/5941F948/5941E011" Ref="#PWR041"  Part="1"
-F 0 "#PWR036" H 5100 2350 50  0001 C CNN
+F 0 "#PWR041" H 5100 2350 50  0001 C CNN
 F 1 "GND" H 5100 2450 50  0000 C CNN
 F 2 "" H 5100 2600 50  0000 C CNN
@@
 	4950 2300 5100 2300
 Wire Wire Line
-	4500 2300 4650 2300
+	4400 2300 4650 2300
 $Comp
 L C C5
@@
 AR Path="/5941B2B4/59727314" Ref="#PWR037"  Part="1"
 AR Path="/5941F948/59727314" Ref="#PWR042"  Part="1"
-F 0 "#PWR037" H 6350 2350 50  0001 C CNN
+F 0 "#PWR042" H 6350 2350 50  0001 C CNN
 F 1 "GND" H 6350 2450 50  0000 C CNN
 F 2 "" H 6350 2600 50  0000 C CNN
@@
 	0    1    1    0
 $EndComp
-Text Label 4500 2300 2    60   ~ 0
-3v3f
-Text Label 4000 3350 2    60   ~ 0
-3v3f
-Text Label 5300 3250 2    60   ~ 0
-3v3f
-Text Label 6600 3150 2    60   ~ 0
-3v3f
-Text GLabel 6350 2300 2    60   Input ~ 0
-ref_filter
 Text GLabel 3700 3550 0    60   Input ~ 0
 ref_filter
@@
 Text GLabel 6300 3350 0    60   Input ~ 0
 ref_filter
+Text GLabel 6350 2300 2    60   Input ~ 0
+ref_filter
+$Comp
+L MCP6004 U3
+U 1 1 5941D635
+P 4100 3650
+AR Path="/5941B2B4/5941D635" Ref="U3"  Part="1"
+AR Path="/5941F948/5941D635" Ref="U3"  Part="4"
+F 0 "U3" H 4150 3850 50  0000 C CNN
+F 1 "MCP6004" H 4250 3450 50  0000 C CNN
+F 2 "custom_footprints:DIP-14_W7.62mm_Socket" H 4050 3750 50  0001 C CNN
+F 3 "" H 4150 3850 50  0000 C CNN
+	1    4100 3650
+	1    0    0    -1
+$EndComp
+Text GLabel 4400 2300 0    60   Input ~ 0
+3v3f
+Connection ~ 4500 2300
+Text GLabel 3800 3350 0    60   Input ~ 0
+3v3f
+Wire Wire Line
+	3800 3350 4000 3350
+Text GLabel 5100 3250 0    60   Input ~ 0
+3v3f
+Wire Wire Line
+	5100 3250 5300 3250
+Text GLabel 6400 3150 0    60   Input ~ 0
+3v3f
+Wire Wire Line
+	6400 3150 6600 3150
 $EndSCHEMATC
